File: proves_radio_stick_V2/proves_radio_stick_V2.kicad_sch (KiCad schematic)
At the start: 77 parts, among them J1 SWD Port, J12 USB_C_Receptacle_USB2.0_16P, J2 Conn_Coaxial, J22 SWD Port, J3 Screw_Terminal_01x10, J4 Conn_01x06_Pin, SW1 KMR2, SW2 KMR2, U11 W25Q128JVS, U18 RP2350_60QFN, U2 TPS62085RLTT, U3 E22-400M30S, Y1 ABM8-272-T3

Commit message: V2: add TPS22918 soft-start switch on RF_VCC, drop J1
Limits USB plug-in inrush: the 110 uF radio bulk now sits behind U19
(CT 1 nF, ~2.9 ms ramp, ~0.19 A peak) so the host sees ~11 uF. GPIO18
drives the enable via RF_PWR_EN; R95 10k to 3V3 keeps the radio on by
default. Removed the 2.54 mm SWD header J1 (duplicate of JST J22) to
free routing for the enable line.

Co-Authored-By: Claude Fable 5.1 <noreply@anthropic.com>
Claude-Session: https://claude.ai/code/session_01N2AhKET2rgFbanw1Dr874g
Parts:
- removed J1: SWD Port, Connector_PinHeader_2.54mm:PinHeader_1x03_P2.54mm_Vertical, symbol Connector_Generic:Conn_01x03
- added C79: 1nF, Capacitor_SMD:C_0402_1005Metric, symbol Device:C
- added C80: 1uF, Capacitor_SMD:C_0402_1005Metric, symbol Device:C
- added R95: 10k, Resistor_SMD:R_0402_1005Metric, symbol Device:R
- added U19: TPS22918DBVR, Package_TO_SOT_SMD:SOT-23-6, symbol easyeda2kicad:TPS22918DBV
Connections:
- net +3V3: now also R95.2
- net GND: now also C79.2, C80.2, U19.2 (GND)
- net RF_VCC: now also U19.5 (QOD), U19.6 (VOUT); no longer FB1.2
- net RF_PWR_EN: now reaches U18.29 (GPIO18)
- net RF_PWR_EN: now also R95.1, U19.3 (ON)
- new net: C79.1, U19.4 (CT)
- new net RF_5V_IN: C80.1, FB1.2, U19.1 (VIN)
- no-connect marks 6 -> 5
Other:
- note added: "U19 TPS22918: CT 1nF -> 2.9 ms ramp, 0.19 A inrush into 110 uF. R95 to +3V3 = radio ON by default; move R95 to GND for default OFF (firmware enables via GPIO18)."
- moved on the sheet: FB1

Commit message: V2: burn down ERC/DRC and schematic-parity items
ERC 4 errors -> 0 (no_connects on GPIO4/5/12/13), warnings 110 -> 45.
DRC 67 -> 48, all remaining are cached-library mismatches; parity 57 -> 0.
Retyped EasyEDA symbol pins, refreshed GND/LED cached symbols, cleared
silk-over-copper and edge items without moving copper, removed a
dangling +1V1 stub and off-board silk text, synced Description and
Datasheet fields, fixed C3/H2-H4 footprint links and R26/R27 BOM flag.

Co-Authored-By: Claude Fable 5.1 <noreply@anthropic.com>
Claude-Session: https://claude.ai/code/session_01N2AhKET2rgFbanw1Dr874g
Parts:
- C3: footprint Capacitor_SMD:C_0603_1608Metric -> Capacitor_SMD:C_0805_2012Metric
- H2, H3, H4: footprint MountingHole:MountingHole_2.2mm_M2_Pad_Via -> MountingHole:MountingHole_2.2mm_M2_Pad_TopBottom
- R26, R27: now in the parts list
Connections:
- no-connect marks 5 -> 9
Changed lines of the file:
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@@
 			)
 		)
-		(property "Footprint" "MountingHole:MountingHole_2.2mm_M2_Pad_Via"
+		(property "Footprint" "MountingHole:MountingHole_2.2mm_M2_Pad_TopBottom"
 			(at 73.66 269.24 0)
 			(effects
@@
 			)
 		)
-		(property "Footprint" "Capacitor_SMD:C_0603_1608Metric"
+		(property "Footprint" "Capacitor_SMD:C_0805_2012Metric"
 			(at 295.6052 160.02 0)
 			(effects
@@
 			)
 		)
-		(property "Footprint" "MountingHole:MountingHole_2.2mm_M2_Pad_Via"
+		(property "Footprint" "MountingHole:MountingHole_2.2mm_M2_Pad_TopBottom"
 			(at 73.66 274.32 0)
 			(effects
@@
 			)
 		)
-		(property "Footprint" "MountingHole:MountingHole_2.2mm_M2_Pad_Via"
+		(property "Footprint" "MountingHole:MountingHole_2.2mm_M2_Pad_TopBottom"
 			(at 73.66 279.4 0)
 			(effects
@@
 		(unit 1)
 		(exclude_from_sim no)
-		(in_bom no)
+		(in_bom yes)
 		(on_board yes)
 		(dnp no)
@@
 		(unit 1)
 		(exclude_from_sim no)
-		(in_bom no)
+		(in_bom yes)
 		(on_board yes)
 		(dnp no)
@@
 		(at 210.82 121.92)
 	)
+	(no_connect
+		(at 210.82 83.82)
+	)
+	(no_connect
+		(at 210.82 86.36)
+	)
+	(no_connect
+		(at 210.82 104.14)
+	)
+	(no_connect
+		(at 210.82 106.68)
+	)
 	(symbol
