File: proves_radio_stick_V2/proves_radio_stick_V2.kicad_sch (KiCad schematic)
At the start: 80 parts, among them J12 USB_C_Receptacle_USB2.0_16P, J2 Conn_Coaxial, J22 SWD Port, J3 Screw_Terminal_01x10, J4 Conn_01x06_Pin, SW1 KMR2, SW2 KMR2, U11 W25Q128JVS, U18 RP2350_60QFN, U19 TPS22918DBVR, U2 TPS62085RLTT, U3 E22-400M30S, Y1 ABM8-272-T3

Commit message: V2: source J3 terminal block, DNP J4/TP1-7, prune dead lib rows
J3 gets LCSC C474928 (Cixi Kefa KF128-2.54-10P, drop-in for the Phoenix
MPT 0,5/10-2,54 footprint, 1.1 mm drills). J4 header and TP1-TP7 marked
exclude-from-BOM so schematic, BOM and CPL agree. Removed lib-table rows
pointing at directories that no longer exist. Production files
regenerated from this state.

Co-Authored-By: Claude Fable 5.1 <noreply@anthropic.com>
Claude-Session: https://claude.ai/code/session_01N2AhKET2rgFbanw1Dr874g
Parts:
- J3: LCSC Part (none) -> C474928; MPN (none) -> KF128-2.54-10P
- J4, TP1, TP2, TP3, TP4, TP5, TP6, TP7: now left out of the parts list
Changed lines of the file:
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@@
 		(unit 1)
 		(exclude_from_sim no)
-		(in_bom yes)
+		(in_bom no)
 		(on_board yes)
 		(dnp no)
@@
 		(unit 1)
 		(exclude_from_sim no)
-		(in_bom yes)
+		(in_bom no)
 		(on_board yes)
 		(dnp no)
@@
 		(unit 1)
 		(exclude_from_sim no)
-		(in_bom yes)
+		(in_bom no)
 		(on_board yes)
 		(dnp no)
@@
 		(unit 1)
 		(exclude_from_sim no)
-		(in_bom yes)
+		(in_bom no)
 		(on_board yes)
 		(dnp no)
@@
 			)
 		)
+		(property "LCSC Part" "C474928"
+			(at 372.11 219.71 0)
+			(effects
+				(font
+					(size 1.27 1.27)
+				)
+				(hide yes)
+			)
+		)
+		(property "MPN" "KF128-2.54-10P"
+			(at 372.11 219.71 0)
+			(effects
+				(font
+					(size 1.27 1.27)
+				)
+				(hide yes)
+			)
+		)
 		(property "Datasheet" "~"
 			(at 372.11 219.71 0)
@@
 		(unit 1)
 		(exclude_from_sim no)
-		(in_bom yes)
+		(in_bom no)
 		(on_board yes)
 		(dnp no)
@@
 		(unit 1)
 		(exclude_from_sim no)
-		(in_bom yes)
+		(in_bom no)
 		(on_board yes)
 		(dnp no)
@@
 		(unit 1)
 		(exclude_from_sim no)
-		(in_bom yes)
+		(in_bom no)
 		(on_board yes)
 		(dnp no)
@@
 		(unit 1)
 		(exclude_from_sim no)
-		(in_bom yes)
+		(in_bom no)
 		(on_board yes)
 		(dnp no)

Commit message: V2: rearrange schematic right half for readability
Buck, radio 5 V rail, radio, antenna/ESD and connector blocks moved
into three rows with section titles; overlapping reference, value,
PWR_FLAG and note text separated. Rigid block moves only; netlist
identical to previous commit.

Co-Authored-By: Claude Fable 5.1 <noreply@anthropic.com>
Claude-Session: https://claude.ai/code/session_01N2AhKET2rgFbanw1Dr874g
Other:
- note added: "3.3 V Buck"
- note added: "Antenna / ESD"
- note added: "Connectors"
- note added: "RP2350"
- note added: "Radio 5 V Rail"
- note added: "Radio E22-400M30S"
- note added: "USB-C"
- moved on the sheet: C1, C14, C15, C3, C4, C5, C6, C7, C79, C80, FB1, J2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

Commit message: V2: JLCPCB parts database and LCSC fields on every part
Adds jlcpcb/project.db for the kicad-jlcpcb-tools plugin (81 rows, live
stock), LCSC Part on all 52 previously blank symbols and footprints,
exclude-from-pos on the hand-fit J4/TP1-7, and moves C4 to C84455
(Murata GRM32ER61A107ME20L, a true 1210 10 V part; C15008 is 1206
6.3 V per JLC). Board and project files are now in KiCad 10 format
after a GUI save.

Co-Authored-By: Claude Fable 5.1 <noreply@anthropic.com>
Claude-Session: https://claude.ai/code/session_01N2AhKET2rgFbanw1Dr874g
Parts:
- C1, C2, C67, C70, C71, C72, C73, C74, C76, C77, C78: LCSC Part (none) -> C1525
- C14: LCSC Part (none) -> C59461
- C15, C75: LCSC Part (none) -> C19702
- C3: LCSC Part (none) -> C16780
- C4: LCSC Part C15008 -> C84455
- C63, C64: LCSC Part (none) -> C1548
- C65, C66, C68, C69: LCSC Part (none) -> C23733
- D1, D3: LCSC Part (none) -> C2290
- D4: LCSC Part (none) -> C48192
- J12: LCSC Part (none) -> C165948
- J2: LCSC Part (none) -> C3174425
- J22: LCSC Part (none) -> C160389
- L3: LCSC Part (none) -> C42411119
- R1, R11, R12, R2, R39, R41, R5, R9: LCSC Part (none) -> C25744
- R10, R13, R80, R93: LCSC Part (none) -> C11702
- R26, R27: LCSC Part (none) -> C25905
- R3: LCSC Part (none) -> C54068
- R4: LCSC Part (none) -> C11616
- R7, R8: LCSC Part (none) -> C25092
- R94: LCSC Part (none) -> C25105
- SW1, SW2: LCSC Part (none) -> C72443
- U11: LCSC Part (none) -> C97521
- U18: LCSC Part (none) -> C42411118
- Y1: LCSC Part (none) -> C20625731
