File: proves_radio_stick_V2/proves_radio_stick_V2.kicad_pcb (KiCad board)
At the start: 4 copper layers, 80.5 x 32.9 mm, 78 parts, among them J1 SWD Port, J12 USB_C_Receptacle_USB2.0_16P, J2 Conn_Coaxial, J22 SWD Port, J3 Screw_Terminal_01x10, J4 Conn_01x06_Pin, SW1 KMR2, SW2 KMR2, U11 W25Q128JVS, U18 RP2350_60QFN, U2 TPS62085RLTT, U3 E22-400M30S, Y1 ABM8-272-T3

Commit message: V2: add TPS22918 soft-start switch on RF_VCC, drop J1
Limits USB plug-in inrush: the 110 uF radio bulk now sits behind U19
(CT 1 nF, ~2.9 ms ramp, ~0.19 A peak) so the host sees ~11 uF. GPIO18
drives the enable via RF_PWR_EN; R95 10k to 3V3 keeps the radio on by
default. Removed the 2.54 mm SWD header J1 (duplicate of JST J22) to
free routing for the enable line.

Co-Authored-By: Claude Fable 5.1 <noreply@anthropic.com>
Claude-Session: https://claude.ai/code/session_01N2AhKET2rgFbanw1Dr874g
Parts:
- removed J1: SWD Port, Connector_PinHeader_2.54mm:PinHeader_1x03_P2.54mm_Vertical
- added C79: 1nF, Capacitor_SMD:C_0402_1005Metric, B.Cu at (201.2, 112.5)
- added C80: 1uF, Capacitor_SMD:C_0402_1005Metric, B.Cu at (204.9, 116.3)
- added R95: 10k, Resistor_SMD:R_0402_1005Metric, B.Cu at (201.2, 114.9)
- added U19: TPS22918DBVR, Package_TO_SOT_SMD:SOT-23-6, B.Cu at (204.1, 113.6)
Connections:
- FB1 pad 2: RF_VCC -> RF_5V_IN
- U18 pad 29: unconnected-(U18-GPIO18-Pad29) -> RF_PWR_EN
Routing:
- net RF_PWR_EN: track 0.00 -> 42.1 mm, vias 0 -> 1
- net SWCLK: track 27.1 -> 19.5 mm, vias 1 -> 2
- net RF_5V_IN: track 0.00 -> 5.74 mm, vias 0 -> 1
- net GND: track 84.0 -> 86.6 mm, vias 158 -> 157
- net Net-(U19-CT): track 0.00 -> 1.47 mm
- net SWDIO: track 15.8 -> 14.6 mm, vias 1 -> 2
- net RF_VCC: track 10.6 -> 11.5 mm
- net +3V3: track 62.0 -> 62.4 mm, vias 29 -> 30

Commit message: V2: burn down ERC/DRC and schematic-parity items
ERC 4 errors -> 0 (no_connects on GPIO4/5/12/13), warnings 110 -> 45.
DRC 67 -> 48, all remaining are cached-library mismatches; parity 57 -> 0.
Retyped EasyEDA symbol pins, refreshed GND/LED cached symbols, cleared
silk-over-copper and edge items without moving copper, removed a
dangling +1V1 stub and off-board silk text, synced Description and
Datasheet fields, fixed C3/H2-H4 footprint links and R26/R27 BOM flag.

Co-Authored-By: Claude Fable 5.1 <noreply@anthropic.com>
Claude-Session: https://claude.ai/code/session_01N2AhKET2rgFbanw1Dr874g
Other:
- board text removed: "Wait its all open source?"
